File: entrega2/esquemático/arquivos_kicad/esquematico.kicad_sch (KiCad schematic)
At the start: 10 parts, among them J1 Encoder E2-Q2, J2 Barra de pinos fêmea 1x8, J3 L298N, J4 Barra de pinos fêmea 1x6, J5 Barra de pinos fêmea 1x6, J6 Encoder E2-Q2, J7 ESP32 C3 Super MIni, J8 Barra de pinos fêmea 1x8, M1 Motor TT, M2 Motor TT

Commit message: Atualizei o esquemático e o ReadME.
Parts:
- removed J2, J8: Barra de pinos fêmea 1x8, symbol Connector:Conn_01x08_Pin
- removed J4, J5: Barra de pinos fêmea 1x6, symbol Connector:Conn_01x06_Pin
- added C1, C2: (no value), symbol ProjetoBixo:Barra_de_pinos_2x4
- added C3: 4.7 uF 16V, symbol Device:C
- added C4, C5: (no value), symbol ProjetoBixo:Barra_de_pinos_1x8
- added SW1: Interruptor, symbol Switch:SW_DPST_x2
Connections:
- net 12V: now also SW1.1 (A); no longer J3.3 (12V)
- net 5V: now also C2.8, C3.1
- net GND: now also C1.8, C3.2
- net at J6.1 (D1): now also C4.14; no longer J7.14 (GPIO7)
- net at J6.2 (D2): now also C4.13; no longer J7.13 (GPIO8)
- net at J3.10 (1N4): now also C4.9; no longer J7.9 (GPIO21)
- net at J3.7 (1N1): now also C4.12; no longer J7.12 (GPIO9)
- net at J3.8 (1N2): now also C4.11; no longer J7.11 (GPIO10)
- net at J3.9 (1N3): now also C4.10; no longer J7.10 (GPIO20)
- net at J7.2 (GND): now also C5.15
- net at J7.1 (5V): now also C5.16
- net at J7.16 (GPIO5): now also C4.1; no longer J1.1 (D1)
- net at J1.2 (D2): now also C4.15; no longer J7.15 (GPIO6)
- net at J7.3 (3.3V): now also C5.14
- net at J7.4 (GPIO4): now also C5.13
- net at J7.5 (GPIO3): now also C5.12
- net at J7.6 (GPIO2): now also C5.11
- net at J7.7 (GPIO1): now also C5.10
- net at J7.8 (GPIO0): now also C5.9
- new net: J3.3 (12V), SW1.2 (B)
- new net: C4.16, J1.1 (D1)
- new net: C4.2, J7.15 (GPIO6)
- new net: C4.3, J7.14 (GPIO7)
- new net: C4.4, J7.13 (GPIO8)
- new net: C4.5, J7.12 (GPIO9)
- new net: C4.6, J7.11 (GPIO10)
- new net: C4.7, J7.10 (GPIO20)
- new net: C4.8, J7.9 (GPIO21)
- new net: C2.1, C5.1
- new net: C1.1, C5.2
